File: KiCad/Starter/CDR3585.kicad_pcb (KiCad board)
At the start: 2 copper layers, 114.3 x 88.9 mm, 51 parts, among them J1 AudioJack, J2 Speaker, J3 UART1, J4 Pot, J5 Conn_01x08_Pin, J6 GND, J7 DACOUT, SW1 UP, SW2 LEFT, SW3 DOWN, SW4 RGHT, U1 Adafruit ST7735R, U2 LP-MSPM0G3507, U3 MCP34119P, U4 HiLetGo_ST7735R, U5 ULN2003B, U6 TSOP31438

Commit message: project finsihed need review
Parts:
- removed C4: 0.1uF, ECE319K:C_Axial_200mil
- removed D4: LED, ECE319K:LED_D5.0mm
- removed J5: Conn_01x08_Pin, Connector_PinSocket_2.54mm:PinSocket_1x08_P2.54mm_Vertical
- removed R18: 220, ECE319K:R_Axial_DIN0204_L3.6mm_D1.6mm_P7.62mm_Horizontal
- removed R7, R8: 1.5k, ECE319K:R_Axial_DIN0204_L3.6mm_D1.6mm_P7.62mm_Horizontal
- removed U4: HiLetGo_ST7735R, ECE319K:hiletgo_st7735r
- removed U5: ULN2003B, ECE319K:DIP-16_W7.62mm
- removed U6: TSOP31438, ECE319K:TSOP31438
- added D5: LED, ECE319K:LED_D5.0mm, F.Cu at (85.0, 50.5)
- added D6: LED, ECE319K:LED_D5.0mm, F.Cu at (85.0, 63.5)
- added D7: LED, ECE319K:LED_D5.0mm, F.Cu at (85.0, 76.0)
- added J8: Joystick, ECE319K:SparkfunJoystick, F.Cu at (136.3, 111.8)
- added R19: 470, ECE319K:R_Axial_DIN0204_L3.6mm_D1.6mm_P7.62mm_Horizontal, F.Cu at (80.9, 58.0)
- added R20: 470, ECE319K:R_Axial_DIN0204_L3.6mm_D1.6mm_P7.62mm_Horizontal, F.Cu at (81.4, 71.0)
- added R21: 470, ECE319K:R_Axial_DIN0204_L3.6mm_D1.6mm_P7.62mm_Horizontal, F.Cu at (80.9, 83.5)
- added R22: 12k, ECE319K:R_Axial_DIN0204_L3.6mm_D1.6mm_P7.62mm_Horizontal, F.Cu at (68.4, 66.5)
- added R23: 12k, ECE319K:R_Axial_DIN0204_L3.6mm_D1.6mm_P7.62mm_Horizontal, F.Cu at (68.4, 70.5)
- J1: value AudioJack -> Joystick; footprint ECE319K:Jack_3.5mm_CUI_SJ1-3523N_Horizontal -> ECE319K:SparkfunJoystick
- moved U1 146.4 mm to (107.0, 77.0)
- moved SW4 127.7 mm to (149.2, 78.2)
- moved R13 125.2 mm to (136.5, 60.0)
- moved R12 124.6 mm to (136.5, 56.0)
- moved R14 123.9 mm to (136.5, 52.0)
- moved R15 116.6 mm to (136.5, 48.0)
- moved SW1 111.7 mm to (139.2, 69.8)
- moved SW2 101.7 mm to (128.8, 78.8)
- moved SW3 97.6 mm to (139.8, 86.2)
- moved RV1 84.0 mm to (90.6, 118.2)
- moved D2 75.0 mm to (104.0, 43.5)
- moved R1 72.2 mm to (99.0, 47.3)
- moved D3 71.0 mm to (117.0, 43.4)
- moved J1 70.6 mm to (61.8, 113.3), turned to 0 degrees
- moved D1 70.3 mm to (91.5, 43.5)
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Connections:
- C1 pad 1: unconnected-(C1-Pad1) -> Net-(U3-FC1)
- C1 pad 2: unconnected-(C1-Pad2) -> GND
- C2 pad 1: unconnected-(C2-Pad1) -> Net-(U3-FC2)
- C2 pad 2: unconnected-(C2-Pad2) -> GND
- C3 pad 1: unconnected-(C3-Pad1) -> DACOUT
- C3 pad 2: unconnected-(C3-Pad2) -> Net-(C3-Pad2)
- D1 pad 1: unconnected-(D1-K-Pad1) -> GND
- D1 pad 2: unconnected-(D1-A-Pad2) -> Net-(D1-A)
- D2 pad 1: unconnected-(D2-K-Pad1) -> GND
- D2 pad 2: unconnected-(D2-A-Pad2) -> Net-(D2-A)
- D3 pad 1: unconnected-(D3-K-Pad1) -> GND
- D3 pad 2: unconnected-(D3-A-Pad2) -> Net-(D3-A)
- J2 pad 1: unconnected-(J2-Pad1) -> Net-(U3-VO1)
- J2 pad 2: unconnected-(J2-Pad2) -> Net-(U3-VO2)
- J4 pad 1: unconnected-(J4-A-Pad1) -> PB18
- J4 pad 2: unconnected-(J4-B-Pad2) -> PB18
- J7 pad 1: unconnected-(J7-A-Pad1) -> DACOUT
- J7 pad 2: unconnected-(J7-B-Pad2) -> DACOUT
- JP1 pad 1: unconnected-(JP1-A-Pad1) -> DACOUT
- JP1 pad 3: unconnected-(JP1-B-Pad3) -> PB18
- R1 pad 1: unconnected-(R1-Pad1) -> PA17
- R1 pad 2: unconnected-(R1-Pad2) -> Net-(D1-A)
- R10 pad 1: unconnected-(R10-Pad1) -> DACOUT
- R10 pad 2: unconnected-(R10-Pad2) -> PB2
- R11 pad 1: unconnected-(R11-Pad1) -> DACOUT
- R11 pad 2: unconnected-(R11-Pad2) -> PB1
- R12 pad 1: unconnected-(R12-Pad1) -> PA24
- R12 pad 2: unconnected-(R12-Pad2) -> GND
- R13 pad 1: unconnected-(R13-Pad1) -> PA25
- R13 pad 2: unconnected-(R13-Pad2) -> GND
- R14 pad 1: unconnected-(R14-Pad1) -> PA26
- R14 pad 2: unconnected-(R14-Pad2) -> GND
- R15 pad 1: unconnected-(R15-Pad1) -> PA27
- R15 pad 2: unconnected-(R15-Pad2) -> GND
- R16 pad 1: unconnected-(R16-Pad1) -> Net-(U3-VIN)
- R16 pad 2: unconnected-(R16-Pad2) -> Net-(C3-Pad2)
- R17 pad 1: unconnected-(R17-Pad1) -> Net-(U3-VO1)
- R17 pad 2: unconnected-(R17-Pad2) -> Net-(U3-VIN)
- R2 pad 1: unconnected-(R2-Pad1) -> PA16
- R2 pad 2: unconnected-(R2-Pad2) -> Net-(D2-A)
- R3 pad 1: unconnected-(R3-Pad1) -> PB12
- R3 pad 2: unconnected-(R3-Pad2) -> Net-(D3-A)
- R4 pad 1: unconnected-(R4-Pad1) -> DACOUT
- R4 pad 2: unconnected-(R4-Pad2) -> PB4
- R5 pad 1: unconnected-(R5-Pad1) -> DACOUT
- R5 pad 2: unconnected-(R5-Pad2) -> Net-(R5-Pad2)
- R6 pad 1: unconnected-(R6-Pad1) -> Net-(R5-Pad2)
- R6 pad 2: unconnected-(R6-Pad2) -> PB3
- R9 pad 1: unconnected-(R9-Pad1) -> DACOUT
- R9 pad 2: unconnected-(R9-Pad2) -> PB2
- RV1 pad 1: unconnected-(RV1-Pad1) -> GND
- RV1 pad 2: unconnected-(RV1-Pad2) -> PB18
- RV1 pad 3: unconnected-(RV1-Pad3) -> +3V3
- SW1 pad 1: unconnected-(SW1-Pad1) -> PA24
- SW1 pad 2: unconnected-(SW1-Pad2) -> +3V3
- SW2 pad 1: unconnected-(SW2-Pad1) -> PA25
- SW2 pad 2: unconnected-(SW2-Pad2) -> +3V3
- SW3 pad 1: unconnected-(SW3-Pad1) -> PA26
- SW3 pad 2: unconnected-(SW3-Pad2) -> +3V3
- SW4 pad 1: unconnected-(SW4-Pad1) -> PA27
- SW4 pad 2: unconnected-(SW4-Pad2) -> +3V3
- U3 pad 1: unconnected-(U3-CD-Pad1) -> GND
- U3 pad 2: unconnected-(U3-FC2-Pad2) -> Net-(U3-FC2)
- U3 pad 3: unconnected-(U3-FC1-Pad3) -> Net-(U3-FC1)
- U3 pad 4: unconnected-(U3-VIN-Pad4) -> Net-(U3-VIN)
- U3 pad 5: unconnected-(U3-VO1-Pad5) -> Net-(U3-VO1)
- U3 pad 6: unconnected-(U3-Vcc-Pad6) -> +5V
- U3 pad 7: unconnected-(U3-GND-Pad7) -> GND
- U3 pad 8: unconnected-(U3-VO2-Pad8) -> Net-(U3-VO2)
Routing:
- net GND: track 0.00 -> 344.9 mm
- net +3V3: track 0.00 -> 268.3 mm, vias 0 -> 1
- net PB0: track 0.00 -> 97.4 mm, vias 0 -> 2
- net PB18: track 0.00 -> 94.3 mm, vias 0 -> 1
- net PB19: track 0.00 -> 89.2 mm, vias 0 -> 1
- net PB24: track 0.00 -> 82.4 mm, vias 0 -> 1
- net DACOUT: track 0.00 -> 82.4 mm, vias 0 -> 1
- net PB4: track 0.00 -> 80.2 mm
- net PA28: track 0.00 -> 79.3 mm, vias 0 -> 1
- net PB1: track 0.00 -> 73.3 mm, vias 0 -> 1
- net PB3: track 0.00 -> 71.6 mm, vias 0 -> 1
- net PB12: track 0.00 -> 70.9 mm
- net PA27: track 0.00 -> 68.7 mm, vias 0 -> 1
- net +5V: track 0.00 -> 68.6 mm, vias 0 -> 1
- net PA26: track 0.00 -> 68.3 mm
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Other:
- board text added: "Carlos Rojas, Grant Osinde"
- board text added: "Carlos Rojas, Granty Osinde"
- board text removed: "Your names"
