File: KiCad/Starter/CDR3585.kicad_sch (KiCad schematic)
At the start: 50 parts, among them J1 AudioJack, J2 Speaker, J3 UART1, J4 Pot, J5 Conn_01x08_Pin, J6 GND, J7 DACOUT, SW1 UP, SW2 LEFT, SW3 DOWN, SW4 RGHT, U1 Adafruit ST7735R, U2 LP-MSPM0G3507, U3 MCP34119P, U4 HiLetGo_ST7735R, U5 ULN2003B, U6 TSOP31438

Commit message: project finsihed need review
Parts:
- removed C4: 0.1uF, ECE319K:C_Axial_200mil, symbol ECE319K:C
- removed D4: LED, ECE319K:LED_D5.0mm, symbol ECE319K:OED-EL-1L2
- removed J1: AudioJack, ECE319K:Jack_3.5mm_CUI_SJ1-3523N_Horizontal, symbol ECE319K:HeadphoneJack
- removed J5: Conn_01x08_Pin, Connector_PinSocket_2.54mm:PinSocket_1x08_P2.54mm_Vertical, symbol Connector:Conn_01x08_Pin
- removed R18: 220, ECE319K:R_Axial_DIN0204_L3.6mm_D1.6mm_P7.62mm_Horizontal, symbol ECE319K:R_0.125W
- removed R7, R8: 1.5k, ECE319K:R_Axial_DIN0204_L3.6mm_D1.6mm_P7.62mm_Horizontal, symbol ECE319K:R_0.125W
- removed U4: HiLetGo_ST7735R, ECE319K:hiletgo_st7735r, symbol ECE319K:HiLetGo_ST7735R
- removed U5: ULN2003B, ECE319K:DIP-16_W7.62mm, symbol ECE319K:ULN2003B
- removed U6: TSOP31438, ECE319K:TSOP31438, symbol ECE319K:TSOP31438
- added D5, D6, D7: LED, ECE319K:LED_D5.0mm, symbol ECE319K:LED
- added J1, J8: Joystick, ECE319K:SparkfunJoystick, symbol ECE319K:Joystick_Sparkfun_COM-09032
- added R19, R20, R21: 470, ECE319K:R_Axial_DIN0204_L3.6mm_D1.6mm_P7.62mm_Horizontal, symbol ECE319K:R_0.125W
- added R22, R23: 12k, ECE319K:R_Axial_DIN0204_L3.6mm_D1.6mm_P7.62mm_Horizontal, symbol ECE319K:R_0.125W
Connections:
- net +3V3: now also RV1.3, SW1.2, SW2.2, SW3.2, SW4.2, J1.12 (SEL+), J1.3 (V+), J1.4 (H+), J8.12 (SEL+), J8.3 (V+), J8.4 (H+)
- net +5V: now also U3.6 (Vcc)
- net DACOUT: now also C3.1, J7.1 (A), J7.2 (B), JP1.1 (A), R10.1, R11.1, R4.1, R5.1, R9.1, R23.1
- net GND: now also C1.2, C2.2, D1.1 (K), D2.1 (K), D3.1 (K), R12.2, R13.2, R14.2, R15.2, RV1.1, U3.1 (CD), U3.7 (GND), D5.1 (K), D6.1 (K), D7.1 (K), J1.1 (V-), J1.6 (H-), J8.1 (V-), J8.6 (H-)
- net PA12: now also J8.11 (SEL-)
- net PA16: now also R2.1
- net PA17: now also R1.1
- net PA24: now also R12.1, SW1.1
- net PA25: now also R13.1, SW2.1
- net PA26: now also R14.1, SW3.1
- net PA27: now also R15.1, SW4.1
- net PA28: now also R19.1
- net PA31: now also R20.1
- net PB0: now also R22.2
- net PB1: now also R11.2
- net PB12: now also R3.1
- net PB16: now also J1.11 (SEL-)
- net PB17: now also J1.2 (Vert)
- net PB18: now also J4.1 (A), J4.2 (B), JP1.3 (B), RV1.2
- net PB19: now also J1.5 (Hori)
- net PB2: now also R10.2, R9.2
- net PB20: now also J8.2 (Vert)
- net PB23: now also R21.1
- net PB24: now also J8.5 (Hori)
- net PB3: now also R6.2
- net PB4: now also R4.2
- net at R1.2: now also D1.2 (A)
- net at D3.2 (A): now also R3.2
- net at U3.2 (FC2): now also C2.1
- net at U3.3 (FC1): now also C1.1
- net at U3.4 (VIN): now also R16.1, R17.2
- net at U3.5 (VO1): now also J2.1, R17.1
- net at U3.8 (VO2): now also J2.2
- net at D2.2 (A): now also R2.2
- net at R16.2: now also C3.2
- net at R6.1: now also R5.2
- new net: D5.2 (A), R19.2
- new net: D6.2 (A), R20.2
- new net: D7.2 (A), R21.2
- new net: R22.1, R23.2
Other:
- title: Starter Project Spring 2025 -> Assignment 1, Carlos, Grant
- moved on the sheet: D2, D3, R10, R11, R17, R2, R3, R4, R5, R6, R9
